File: kicad/ass_shield.kicad_pcb (KiCad board)
At the start: 2 copper layers, 80 x 80 mm, 150 parts, among them J1 6-40V, J2 DEBUG, J3 5V, J4 UART2, J5 U.FL, J7 SP, J8 U.FL, M1 CR1220SMD, Q1 BC817, U1 OPiZero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

Commit message: Add files via upload
Parts:
- U1: footprint imm:OPiZero -> imm:OPiZero4
- moved J3 24.0 mm to (121.2, 127.6), turned to 90 degrees
Routing:
- net Net-(C60-Pad2): track 23.5 -> 51.9 mm, vias 1 -> 2
- net 5V: track 387.3 -> 377.8 mm, vias 6 -> 8
Changed lines of the file:
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@@
     (thickness 1.6)
     (drawings 5)
-    (tracks 1653)
+    (tracks 1665)
     (zones 0)
     (modules 150)
@@
   )
   (setup
-    (last_trace_width 0.2)
+    (last_trace_width 1)
     (user_trace_width 0.2)
     (user_trace_width 0.3)
@@
     (uvia_drill 0.3)
   )
-  (module imm:OPiZero (layer F.Cu)
+  (module imm:OPiZero4 (layer F.Cu)
     (at 77 124)
     (fp_text reference U1 (at 25.4 -43.18) (layer F.SilkS)
@@
     (pad "" thru_hole circle (at 3 -3) (size 4 4) (drill 3) (layers *.Cu *.Mask F.SilkS))
     (pad "" thru_hole circle (at 43 -3) (size 4 4) (drill 3) (layers *.Cu *.Mask F.SilkS))
-    (model /home/user/kicad/libraries/imm_lib/Orange_Pi_Zero_v1_1___Ensamblaje_cp.wrl
-      (offset (xyz 23 25.8 -71))
-      (scale (xyz 1 1 1))
-      (rotate (xyz 0 0 -90))
-    )
     (model ${KISYS3DMOD}/Connector_PinSocket_2.54mm.3dshapes/PinSocket_1x13_P2.54mm_Vertical.wrl
       (offset (xyz 1.5 39 -1.6))
@@
       (rotate (xyz 0 180 0))
     )
-    (model ${KISYS3DMOD}/Connector_PinSocket_2.54mm.3dshapes/PinSocket_1x13_P2.54mm_Vertical.wrl
-      (offset (xyz 1.5 39 -8.5))
-      (scale (xyz 1 1 1))
-      (rotate (xyz 0 180 0))
-    )
     (model ${KISYS3DMOD}/Connector_PinSocket_2.54mm.3dshapes/PinSocket_2x13_P2.54mm_Vertical.wrl
       (offset (xyz 42.2 39 -1.6))
@@
       (rotate (xyz 0 180 0))
     )
-    (model ${KISYS3DMOD}/Connector_PinSocket_2.54mm.3dshapes/PinSocket_2x13_P2.54mm_Vertical.wrl
-      (offset (xyz 42.2 39 -8.5))
-      (scale (xyz 1 1 1))
-      (rotate (xyz 0 180 0))
-    )
   )
   (module imm:cr1220_smd (layer B.Cu)
@@
     (tags "Surface mounted pin header SMD 1x02 2.54mm single row style1 pin1 left")
     (attr smd)
-    (fp_text reference J1 (at 0 3.6 270) (layer B.SilkS)
+    (fp_text reference J1 (at 2.445 -0.07) (layer B.SilkS)
       (effects (font (size 1 1) (thickness 0.15)) (justify mirror))
     )
@@
   )
   (module Connector_PinHeader_2.54mm:PinHeader_1x02_P2.54mm_Vertical_SMD_Pin1Left (layer B.Cu)
-    (at 99.255 117.73 180)
+    (at 121.17 127.555 90)
     (descr "surface-mounted straight pin header, 1x02, 2.54mm pitch, single row, style 1 (pin 1 left)")
     (tags "Surface mounted pin header SMD 1x02 2.54mm single row style1 pin1 left")
     (attr smd)
-    (fp_text reference J3 (at 0.055 -3.47 180) (layer B.SilkS)
+    (fp_text reference J3 (at -2.545 0.13 180) (layer B.SilkS)
       (effects (font (size 1 1) (thickness 0.15)) (justify mirror))
     )
-    (fp_text value 5V (at 0 -3.6 180) (layer B.Fab)
+    (fp_text value 5V (at 0 -3.6 90) (layer B.Fab)
       (effects (font (size 1 1) (thickness 0.15)) (justify mirror))
     )
-    (fp_text user %R (at 0 0 90) (layer B.Fab)
+    (fp_text user %R (at 0 0) (layer B.Fab)
       (effects (font (size 1 1) (thickness 0.15)) (justify mirror))
     )
@@
     (fp_line (start -0.32 2.54) (end 1.27 2.54) (layer B.Fab) (width 0.1))
     (fp_line (start 1.27 -2.54) (end -1.27 -2.54) (layer B.Fab) (width 0.1))
-    (pad 2 smd rect (at 1.655 -1.27 180) (size 2.51 1) (layers B.Cu B.Paste B.Mask)
+    (pad 2 smd rect (at 1.655 -1.27 90) (size 2.51 1) (layers B.Cu B.Paste B.Mask)
       (net 42 5V))
-    (pad 1 smd rect (at -1.655 1.27 180) (size 2.51 1) (layers B.Cu B.Paste B.Mask)
+    (pad 1 smd rect (at -1.655 1.27 90) (size 2.51 1) (layers B.Cu B.Paste B.Mask)
       (net 127 "Net-(C60-Pad2)"))
     (model ${KISYS3DMOD}/Connector_PinHeader_2.54mm.3dshapes/PinHeader_1x02_P2.54mm_Vertical_SMD_Pin1Left.wrl
@@
   (module imm:usb_f2 (layer B.Cu)
     (at 73.4 82.8)
-    (fp_text reference X1 (at -1 8.5) (layer B.SilkS)
+    (fp_text reference X1 (at -1 8.7) (layer B.SilkS)
       (effects (font (size 1 1) (thickness 0.15)) (justify mirror))
     )
@@
   (segment (start 127.300001 80.171283) (end 131.10897 83.980252) (width 0.5) (layer F.Cu) (net 42))
   (segment (start 119.9 70.771282) (end 127.300001 78.171283) (width 0.5) (layer F.Cu) (net 42))
-  (segment (start 97.6 123.4) (end 94 127) (width 1) (layer B.Cu) (net 42))
-  (segment (start 97.6 119) (end 97.6 123.4) (width 1) (layer B.Cu) (net 42))
   (segment (start 114.440451 131.678718) (end 115.406476 131.678718) (width 1) (layer F.Cu) (net 42))
   (segment (start 101.421282 131.678718) (end 114.440451 131.678718) (width 1) (layer F.Cu) (net 42))
@@
   (segment (start 97.55 135.3) (end 97.8 135.3) (width 1) (layer F.Cu) (net 42))
   (segment (start 127.15 118.55) (end 127.3 118.55) (width 1) (layer F.Cu) (net 42))
-  (segment (start 115.406476 130.293524) (end 127.15 118.55) (width 1) (layer F.Cu) (net 42))
+  (segment (start 115.406476 130.293524) (end 119.9 125.8) (width 1) (layer F.Cu) (net 42))
   (segment (start 115.406476 131.678718) (end 115.406476 130.293524) (width 1) (layer F.Cu) (net 42))
   (segment (start 127.3 118.55) (end 127.3 118.4) (width 0.5) (layer F.Cu) (net 42))
@@
   (segment (start 83.090957 116.049999) (end 89.589999 116.049999) (width 0.5) (layer B.Cu) (net 42))
   (segment (start 90.040001 116.500001) (end 90.94 117.4) (width 0.5) (layer B.Cu) (net 42))
+  (segment (start 119.9 125.8) (end 127.15 118.55) (width 1) (layer F.Cu) (net 42))
+  (via (at 119.9 125.8) (size 0.5) (drill 0.3) (layers F.Cu B.Cu) (net 42))
+  (segment (start 119.9 125.8) (end 119.9 125.8) (width 1) (layer F.Cu) (net 42))
+  (via (at 119.9 125.8) (size 0.5) (drill 0.3) (layers F.Cu B.Cu) (net 42))
   (segment (start 84.3 86.17478) (end 84.34994 86.22472) (width 0.2) (layer F.Cu) (net 43))
   (segment (start 84.34994 84.77994) (end 83.27 83.7) (width 0.2) (layer F.Cu) (net 43))
@@
   (segment (start 95.4 82.77) (end 95.875 82.77) (width 0.2) (layer F.Cu) (net 126))
   (segment (start 101.6696 116.9) (end 101.0696 116.3) (width 0.7) (layer F.Cu) (net 127))
-  (segment (start 107 116.9) (end 101.6696 116.9) (width 0.7) (layer F.Cu) (net 127))
+  (segment (start 107 116.9) (end 102.2 116.3) (width 0.7) (layer F.Cu) (net 127))
   (segment (start 97.89998 117.36962) (end 98.9696 116.3) (width 0.2) (layer F.Cu) (net 127))
   (segment (start 98.9696 116.3) (end 101.0696 116.3) (width 0.2) (layer F.Cu) (net 127))
@@
   (segment (start 101.0696 116.3) (end 101.0696 116.3) (width 0.7) (layer F.Cu) (net 127))
   (via (at 101.0696 116.3) (size 0.5) (drill 0.3) (layers F.Cu B.Cu) (net 127))
+  (segment (start 120.94 129.21) (end 120.93 129.2) (width 1) (layer B.Cu) (net 127))
+  (segment (start 122.44 129.21) (end 120.94 129.21) (width 1) (layer B.Cu) (net 127))
+  (segment (start 120.93 129.2) (end 119 129.2) (width 1) (layer B.Cu) (net 127))
+  (segment (start 108.456002 116.3) (end 103.1696 116.3) (width 1) (layer B.Cu) (net 127))
+  (segment (start 103.1696 116.3) (end 101.0696 116.3) (width 1) (layer B.Cu) (net 127))
+  (segment (start 117.599999 125.443997) (end 108.456002 116.3) (width 1) (layer B.Cu) (net 127))
+  (segment (start 117.599999 127.799999) (end 117.599999 125.443997) (width 1) (layer B.Cu) (net 127))
+  (segment (start 119 129.2) (end 117.599999 127.799999) (width 1) (layer B.Cu) (net 127))
+  (segment (start 102.2 116.3) (end 101.6696 116.9) (width 0.7) (layer F.Cu) (net 127))
+  (via (at 102.2 116.3) (size 0.5) (drill 0.3) (layers F.Cu B.Cu) (net 127))
   (via (at 93.5 75.25) (size 0.5) (drill 0.3) (layers F.Cu B.Cu) (net 128))
   (segment (start 80.446019 75.149979) (end 93.399979 75.149979) (width 0.2) (layer B.Cu) (net 128))
@@
     (polygon
       (pts
-        (xy 54.65 56) (xy 146.4 57.85) (xy 139.6 152.95) (xy 54.3 141.75)
+        (xy 57.111 55.242065) (xy 148.861 57.092065) (xy 142.061 152.192065) (xy 56.761 140.992065)
       )
     )
@@
     (polygon
       (pts
-        (xy 55.65 54.45) (xy 148.1 58.3) (xy 140.6 152.4) (xy 56.35 141.2)
+        (xy 57.717368 54.201685) (xy 150.167368 58.051685) (xy 142.667368 152.151685) (xy 58.417368 140.951685)
       )
     )

Commit message: Add files via upload
Parts:
- added J6: i2s, Connector_PinSocket_2.54mm:PinSocket_1x03_P2.54mm_Vertical, B.Cu at (105.0, 83.4)
Connections:
- D29 pad 31: P4 -> Net-(D29-Pad31)
- D29 pad 32: P3 -> Net-(D29-Pad32)
- D29 pad 33: P2 -> Net-(D29-Pad33)
- U1 pad 10: Net-(U1-Pad10) -> (no net)
- U1 pad 202: Net-(U1-Pad202) -> (no net)
- U1 pad 203: Net-(U1-Pad203) -> (no net)
- U1 pad 9: Net-(U1-Pad9) -> (no net)
- U5 pad 6: P2 -> (no net)
- U5 pad 7: P3 -> (no net)
- U5 pad 9: P4 -> (no net)
Routing:
- net Net-(D29-Pad33): track 0.00 -> 23.1 mm, vias 0 -> 1
- net Net-(D29-Pad32): track 0.00 -> 21.1 mm, vias 0 -> 1
- net Net-(D29-Pad31): track 0.00 -> 18.4 mm, vias 0 -> 1
- net P4: track 4.30 -> 0.00 mm
- net P3: track 3.56 -> 0.00 mm
- net P2: track 3.54 -> 0.00 mm
- net GND: vias 126 -> 127
