File: kicad/ass_shield.kicad_pcb (KiCad board)
At the start: 2 copper layers, 80 x 80 mm, 151 parts, among them J1 6-40V, J2 DEBUG, J3 5V, J4 UART2, J5 U.FL, J6 i2s, J7 SP, J8 U.FL, M1 CR1220SMD, Q1 BC817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

Commit message: Add files via upload
Changed lines of the file:
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@@
     (fp_line (start -1.50876 0.98806) (end 1.50876 0.98806) (layer F.SilkS) (width 0.2032))
     (fp_line (start -1.50876 -3.0099) (end -1.50876 0.98806) (layer F.SilkS) (width 0.2032))
-    (pad "" thru_hole circle (at 0 0 105) (size 1.5 1.5) (drill 1.5) (layers *.Cu *.Mask))
+    (pad "" np_thru_hole circle (at 0 0 105) (size 1.5 1.5) (drill 1.5) (layers *.Cu *.Mask))
     (pad 7 smd rect (at 1.22936 -0.05842 105) (size 0.34798 1.89992) (layers F.Cu F.Paste F.Mask))
     (pad 6 smd rect (at -1.22936 -0.05842 105) (size 0.34798 1.89992) (layers F.Cu F.Paste F.Mask))
@@
     (fp_line (start -1.50876 0.98806) (end 1.50876 0.98806) (layer F.SilkS) (width 0.2032))
     (fp_line (start -1.50876 -3.0099) (end -1.50876 0.98806) (layer F.SilkS) (width 0.2032))
-    (pad "" thru_hole circle (at 0 0 15) (size 1.5 1.5) (drill 1.5) (layers *.Cu *.Mask))
+    (pad "" np_thru_hole circle (at 0 0 15) (size 1.5 1.5) (drill 1.5) (layers *.Cu *.Mask))
     (pad 7 smd rect (at 1.22936 -0.05842 15) (size 0.34798 1.89992) (layers F.Cu F.Paste F.Mask))
     (pad 6 smd rect (at -1.22936 -0.05842 15) (size 0.34798 1.89992) (layers F.Cu F.Paste F.Mask))
@@
     (fp_line (start -1.50876 0.98806) (end 1.50876 0.98806) (layer F.SilkS) (width 0.2032))
     (fp_line (start -1.50876 -3.0099) (end -1.50876 0.98806) (layer F.SilkS) (width 0.2032))
-    (pad "" thru_hole circle (at 0 0 285) (size 1.5 1.5) (drill 1.5) (layers *.Cu *.Mask))
+    (pad "" np_thru_hole circle (at 0 0 285) (size 1.5 1.5) (drill 1.5) (layers *.Cu *.Mask))
     (pad 7 smd rect (at 1.22936 -0.05842 285) (size 0.34798 1.89992) (layers F.Cu F.Paste F.Mask))
     (pad 6 smd rect (at -1.22936 -0.05842 285) (size 0.34798 1.89992) (layers F.Cu F.Paste F.Mask))
@@
     (fp_line (start -1.50876 0.98806) (end 1.50876 0.98806) (layer F.SilkS) (width 0.2032))
     (fp_line (start -1.50876 -3.0099) (end -1.50876 0.98806) (layer F.SilkS) (width 0.2032))
-    (pad "" thru_hole circle (at 0 0 195) (size 1.5 1.5) (drill 1.5) (layers *.Cu *.Mask))
+    (pad "" np_thru_hole circle (at 0 0 195) (size 1.5 1.5) (drill 1.5) (layers *.Cu *.Mask))
     (pad 7 smd rect (at 1.22936 -0.05842 195) (size 0.34798 1.89992) (layers F.Cu F.Paste F.Mask))
     (pad 6 smd rect (at -1.22936 -0.05842 195) (size 0.34798 1.89992) (layers F.Cu F.Paste F.Mask))

Commit message: a msg
Parts:
- AE1, AE2, AE3, AE4: footprint imm:rf_antenna_0.8mm -> Connector_Coaxial:U.FL_Hirose_U.FL-R-SMT-1_Vertical; moved to B.Cu
- C10, C9: value 0,047 µF -> 47 nF
- C17: value 10µF 50V -> 10 µF 50V
- C22: value 100 nF -> 0,1 µF
- C60: value 22µF 6,3V -> 22 µF 6,3V
- D24, D25, D26, D27: value >VALUE -> ADMP421
- R1: value 200 -> 200 R
- R14: value 100 -> 100 R
- R2, R3, R4, R5: value 37 -> 37 R
- U2: footprint Package_SO:SOIC-16W_7.5x10.3mm_P1.27mm -> Package_SO:SO-8_5.3x6.2mm_P1.27mm
- moved U2 2.73 mm to (95.9, 75.9), turned to 180 degrees
- moved AE2 1.17 mm to (102.9, 97.2)
- moved AE1 0.97 mm to (98.7, 97.3), turned to 180 degrees
- moved AE4 0.94 mm to (102.8, 102.4)
- moved AE3 0.72 mm to (98.6, 102.4), turned to 180 degrees
Routing:
- net GND: track 183.3 -> 177.8 mm, vias 127 -> 126
- net Net-(AE1-Pad1): track 5.34 -> 8.59 mm, vias 0 -> 1
- net Net-(AE3-Pad1): track 6.99 -> 10.2 mm, vias 0 -> 1
- net Net-(AE2-Pad1): track 11.4 -> 13.0 mm, vias 0 -> 1
- net 3,3V: track 358.0 -> 358.8 mm
- net Net-(D28-Pad7): track 11.5 -> 12.0 mm
- net Net-(AE4-Pad1): track 5.15 -> 5.18 mm, vias 0 -> 1
Other:
- board text added: "Ass shield v1.0"

Commit message: a msg
Parts:
- added C61: 8.2pF, Capacitor_SMD:C_0402_1005Metric, F.Cu at (101.0, 82.5)
- added C62: 8.2pF, Capacitor_SMD:C_0402_1005Metric, F.Cu at (101.0, 80.7)
- added C63: 270pF, Capacitor_SMD:C_0402_1005Metric, F.Cu at (100.0, 80.7)
- added C64: 270pF, Capacitor_SMD:C_0402_1005Metric, F.Cu at (93.9, 77.8)
- added C65: 10pF, Capacitor_SMD:C_0402_1005Metric, F.Cu at (94.8, 74.1)
- added C66: 0.1uF, Capacitor_SMD:C_0402_1005Metric, F.Cu at (96.1, 70.3)
- added C67: 6.8pF, Capacitor_SMD:C_0402_1005Metric, F.Cu at (92.1, 72.2)
- added C68: 100pF, Capacitor_SMD:C_0402_1005Metric, F.Cu at (95.1, 70.3)
- added C69: 12pF, Capacitor_SMD:C_0402_1005Metric, F.Cu at (93.5, 72.7)
- added C70: 120pF, Capacitor_SMD:C_0402_1005Metric, F.Cu at (95.3, 72.7)
- added C71: 33pF, Capacitor_SMD:C_0402_1005Metric, F.Cu at (94.2, 70.3)
- added C72: 100pF, Capacitor_SMD:C_0402_1005Metric, F.Cu at (101.1, 77.5)
- added C73: 0.1uF, Capacitor_SMD:C_0402_1005Metric, F.Cu at (102.5, 74.8)
- added C74: 1uF, Capacitor_SMD:C_0402_1005Metric, F.Cu at (101.1, 76.4)
- added C75: 4.7pF, Capacitor_SMD:C_0402_1005Metric, F.Cu at (95.8, 76.0)
- added D31: UPG2214TB, Package_TO_SOT_SMD:SOT-23-6, F.Cu at (97.6, 79.0)
- added J9: Conn_Coaxial, Connector_Coaxial:U.FL_Hirose_U.FL-R-SMT-1_Vertical, B.Cu at (96.8, 82.1)
- added L19: 18nH, Inductor_SMD:L_0402_1005Metric, F.Cu at (100.0, 82.5)
- added L20: 24nH, Inductor_SMD:L_0402_1005Metric, F.Cu at (93.9, 76.0)
- added L21: 24nH, Inductor_SMD:L_0402_1005Metric, F.Cu at (92.8, 70.8)
- added L22: 11nH, Inductor_SMD:L_0402_1005Metric, F.Cu at (93.5, 71.8)
- added L23: 270nH, Inductor_SMD:L_0402_1005Metric, F.Cu at (95.3, 71.8)
- added L24: 33nH, Inductor_SMD:L_0402_1005Metric, F.Cu at (95.8, 74.1)
- added R15: 50R, Resistor_SMD:R_0402_1005Metric, F.Cu at (93.9, 74.1)
- added R16: 100k, Resistor_SMD:R_0402_1005Metric, F.Cu at (98.0, 76.3)
- added U7: SI4432-B1-FMR, Package_DFN_QFN:QFN-20-1EP_4x4mm_P0.5mm_EP2.5x2.5mm, F.Cu at (99.2, 73.0)
- added Y8: Crystal_GND24, Crystal:Crystal_SMD_3225-4Pin_3.2x2.5mm, F.Cu at (98.8, 68.3)
- Y6: footprint w_crystal:crystal_tc-38_horiz -> imm:Crystal_SMD_3215-2Pin_3.2x1.5mm; moved to F.Cu
- moved U2 42.1 mm to (129.4, 101.3)
- moved U3 11.2 mm to (109.2, 80.8), turned to 270 degrees
- moved Y6 4.09 mm to (127.7, 96.4)
- moved C29 1.43 mm to (128.6, 94.7)
- moved C30 0.91 mm to (126.7, 94.7)
Connections:
- U1 pad 111: UART2_RX -> NSEL
- U1 pad 113: UART2_TX -> NIRQ
- U1 pad 202: (no net) -> UART2_RX
- U1 pad 203: (no net) -> UART2_TX
Routing:
- net NIRQ: track 0.00 -> 57.9 mm, vias 0 -> 1
- net NSEL: track 0.00 -> 49.8 mm, vias 0 -> 1
- net MISO: track 3.74 -> 44.1 mm
- net SCK: track 4.78 -> 42.8 mm
- net Net-(M1-Pad2): track 101.2 -> 65.6 mm, vias 1 -> 3
- net MOSI: track 8.80 -> 43.4 mm
- net SDA: track 86.6 -> 115.4 mm
- net SCL: track 78.8 -> 107.2 mm
- net UART2_RX: track 11.7 -> 35.3 mm
- net UART2_TX: track 8.40 -> 30.8 mm
- net Net-(C66-Pad2): track 0.00 -> 15.9 mm, vias 0 -> 2
- net P0: track 17.0 -> 31.1 mm
- net Net-(D24-Pad5): track 134.6 -> 148.1 mm, vias 6 -> 8
- net RESET: track 33.4 -> 43.7 mm
- net 3,3V: track 358.8 -> 348.7 mm, vias 21 -> 23
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Other:
- board text added: "+6-40V"
- board text added: "3,3V"
- board text added: "315"
- board text added: "433"
- board text added: "Ass shield v1.1"
- board text added: "BCLK"
- board text added: "DC"
- board text added: "DD"
- board text added: "DEBUG ZIGBEE"
- board text added: "GND"
- board text added: "I2S ADAU1772"
- board text added: "JP DC EXT"
- board text added: "Kusheev Sergei"
- board text added: "L+"
- board text added: "L-"
- board text added: "LRCLK"
- board text added: "NRF24L01+"
- board text added: "R+"
- board text added: "R-"
- board text added: "RECEIVER"
- board text added: "RESET"
- board text added: "RX"
- board text added: "SDATA"
- board text added: "SI4432"
- board text added: "TRANSMITTER"
- board text added: "TX"
- board text added: "UART0 DEBUG"
- board text added: "ZIGBEE"
- board text removed: "Ass shield v1.0"

Commit message: a msg
Parts:
- C22, C32, C33, C34, C35, C40, C42, C44, C46, C49: value 0,1 µF -> 100 nF
- C61, C62: value 8.2pF -> 8,2 pF
- C63, C64: value 270pF -> 270 pF
- C65: value 10pF -> 10 pF
- C66, C73: value 0.1uF -> 100 nF
- C67: value 6.8pF -> 6,8 pF
- C68, C72: value 100pF -> 100 pF
- C69: value 12pF -> 12 pF
- C70: value 120pF -> 120 pF
- C71: value 33pF -> 33 pF
- C74: value 1uF -> 1 µF
- C75: value 4.7pF -> 4,7 pF
- D24, D25, D26, D27: footprint imm:ADMP421 -> imm:ADMP421_2
- L19: value 18nH -> 18 nH
- L20, L21: value 24nH -> 24 nH
- L22: value 11nH -> 11 nH
- L23: value 270nH -> 270 nH
- L24: value 33nH -> 33 nH
Routing:
- net 3,3V: track 348.7 -> 389.5 mm, vias 23 -> 25
- net Net-(D24-Pad5): track 148.1 -> 174.5 mm, vias 8 -> 9
- net CLKD: track 222.3 -> 244.2 mm, vias 4 -> 7
- net Net-(D26-Pad5): track 67.0 -> 79.7 mm, vias 2 -> 3
- net Net-(M1-Pad2): track 65.6 -> 67.3 mm
- net GND: track 173.7 -> 174.7 mm, vias 133 -> 147
