File: kicad/ass_shield.sch (KiCad schematic (older format))
At the start: 151 parts, among them J1 6-40V, J2 DEBUG, J3 5V, J4 UART2, J5 U.FL, J6 i2s, J7 SP, J8 U.FL, M1 CR1220SMD, Q1 BC817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

Commit message: a msg
Parts:
- AE1, AE2, AE3, AE4: footprint imm:rf_antenna_0.8mm -> Connector_Coaxial:U.FL_Hirose_U.FL-R-SMT-1_Vertical; symbol Device:Antenna -> Connector:Conn_Coaxial
- C10, C9: value 0,047 µF -> 47 nF
- C17: value 10µF 50V -> 10 µF 50V
- C22: value 100 nF -> 0,1 µF
- C60: value 22µF 6,3V -> 22 µF 6,3V
- R1: value 200 -> 200 R
- R14: value 100 -> 100 R
- R2, R3, R4, R5: value 37 -> 37 R
- U2: footprint Package_SO:SOIC-16W_7.5x10.3mm_P1.27mm -> Package_SO:SO-8_5.3x6.2mm_P1.27mm
Connections:
- net GND: now also AE1.2 (Ext), AE2.2 (Ext), AE3.2 (Ext), AE4.2 (Ext)
Changed lines of the file:
@@
 	1850 7400 1650 7400
 $Comp
-L Device:Antenna AE4
+L Connector:Conn_Coaxial AE4
 U 1 1 5B6F3B98
 P 650 7350
 F 0 "AE4" V 867 7295 50  0000 C CNN
 F 1 "Antenna" V 776 7295 50  0000 C CNN
-F 2 "imm:rf_antenna_0.8mm" H 650 7350 50  0001 C CNN
+F 2 "Connector_Coaxial:U.FL_Hirose_U.FL-R-SMT-1_Vertical" H 650 7350 50  0001 C CNN
 F 3 "~" H 650 7350 50  0001 C CNN
 	1    650  7350
-	0    -1   -1   0
+	-1   0    0    1
 $EndComp
-Connection ~ 850  7350
 $Comp
 L ass_shield-rescue:syn115-imm_lib D8
@@
 	1850 5950 1650 5950
 $Comp
-L Device:Antenna AE3
+L Connector:Conn_Coaxial AE3
 U 1 1 5B6E4678
 P 650 5900
 F 0 "AE3" V 867 5845 50  0000 C CNN
 F 1 "Antenna" V 776 5845 50  0000 C CNN
-F 2 "imm:rf_antenna_0.8mm" H 650 5900 50  0001 C CNN
+F 2 "Connector_Coaxial:U.FL_Hirose_U.FL-R-SMT-1_Vertical" H 650 5900 50  0001 C CNN
 F 3 "~" H 650 5900 50  0001 C CNN
 	1    650  5900
-	0    -1   -1   0
+	-1   0    0    1
 $EndComp
-Connection ~ 850  5900
 $Comp
 L power:GND #PWR027
@@
 P 1800 5500
 F 0 "C9" H 1915 5546 50  0000 L CNN
-F 1 "0,047 µF" H 1915 5455 50  0000 L CNN
+F 1 "47 nF" H 1915 5455 50  0000 L CNN
 F 2 "Capacitor_SMD:C_0402_1005Metric" V 1650 5450 50  0001 C CNN
 F 3 "" H 1800 5500 50  0001 C CNN
@@
 P 1800 6950
 F 0 "C10" H 1915 6996 50  0000 L CNN
-F 1 "0,047 µF" H 1915 6905 50  0000 L CNN
+F 1 "47 nF" H 1915 6905 50  0000 L CNN
 F 2 "Capacitor_SMD:C_0402_1005Metric" V 1650 6900 50  0001 C CNN
 F 3 "" H 1800 6950 50  0001 C CNN
@@
 5V
 $Comp
-L Device:Antenna AE2
+L Connector:Conn_Coaxial AE2
 U 1 1 5B70D9CD
 P 600 6400
 F 0 "AE2" H 680 6391 50  0000 L CNN
 F 1 "Antenna" H 680 6300 50  0000 L CNN
-F 2 "imm:rf_antenna_0.8mm" H 600 6400 50  0001 C CNN
+F 2 "Connector_Coaxial:U.FL_Hirose_U.FL-R-SMT-1_Vertical" H 600 6400 50  0001 C CNN
 F 3 "~" H 600 6400 50  0001 C CNN
 	1    600  6400
-	1    0    0    -1
+	0    -1   -1   0
 $EndComp
-Connection ~ 600  6600
 $Comp
-L Device:Antenna AE1
+L Connector:Conn_Coaxial AE1
 U 1 1 5B70DA5F
 P 600 4950
 F 0 "AE1" H 680 4941 50  0000 L CNN
 F 1 "Antenna" H 680 4850 50  0000 L CNN
-F 2 "imm:rf_antenna_0.8mm" H 600 4950 50  0001 C CNN
+F 2 "Connector_Coaxial:U.FL_Hirose_U.FL-R-SMT-1_Vertical" H 600 4950 50  0001 C CNN
 F 3 "~" H 600 4950 50  0001 C CNN
 	1    600  4950
-	1    0    0    -1
+	0    -1   -1   0
 $EndComp
-Connection ~ 600  5150
 Text GLabel 1250 1400 0    50   Input ~ 0
 LR
@@
 P 10650 5200
 F 0 "R14" V 10443 5200 50  0000 C CNN
-F 1 "100" V 10534 5200 50  0000 C CNN
+F 1 "100 R" V 10534 5200 50  0000 C CNN
 F 2 "Resistor_SMD:R_0402_1005Metric" V 10550 5250 50  0001 C CNN
 F 3 "" H 10650 5300 50  0001 C CNN
@@
 F 0 "U2" H 4450 5215 50  0000 C CNN
 F 1 "DS3231M" H 4450 5124 50  0000 C CNN
-F 2 "Package_SO:SOIC-16W_7.5x10.3mm_P1.27mm" H 4480 4900 20  0001 C CNN
+F 2 "Package_SO:SO-8_5.3x6.2mm_P1.27mm" H 4480 4900 20  0001 C CNN
 F 3 "" H 4450 4750 50  0001 C CNN
 	1    4450 4750
@@
 P 3900 4200
 F 0 "C17" V 3648 4200 50  0000 C CNN
-F 1 "10µF 50V" V 3739 4200 50  0000 C CNN
+F 1 "10 µF 50V" V 3739 4200 50  0000 C CNN
 F 2 "Capacitor_SMD:C_1206_3216Metric" V 3750 4150 50  0001 C CNN
 F 3 "" H 3900 4200 50  0001 C CNN
@@
 P 5300 3550
 F 0 "C22" V 5048 3550 50  0000 C CNN
-F 1 "100 nF" V 5139 3550 50  0000 C CNN
+F 1 "0,1 µF" V 5139 3550 50  0000 C CNN
 F 2 "Capacitor_SMD:C_0402_1005Metric" V 5150 3500 50  0001 C CNN
 F 3 "" H 5300 3550 50  0001 C CNN
@@
 P 3450 2700
 F 0 "R1" V 3243 2700 50  0000 C CNN
-F 1 "200" V 3334 2700 50  0000 C CNN
+F 1 "200 R" V 3334 2700 50  0000 C CNN
 F 2 "Resistor_SMD:R_0402_1005Metric" V 3380 2700 50  0001 C CNN
 F 3 "~" H 3450 2700 50  0001 C CNN
@@
 P 3800 1150
 F 0 "R2" V 3593 1150 50  0000 C CNN
-F 1 "37" V 3684 1150 50  0000 C CNN
+F 1 "37 R" V 3684 1150 50  0000 C CNN
 F 2 "Resistor_SMD:R_0402_1005Metric" V 3730 1150 50  0001 C CNN
 F 3 "~" H 3800 1150 50  0001 C CNN
@@
 P 3800 1550
 F 0 "R3" V 3593 1550 50  0000 C CNN
-F 1 "37" V 3684 1550 50  0000 C CNN
+F 1 "37 R" V 3684 1550 50  0000 C CNN
 F 2 "Resistor_SMD:R_0402_1005Metric" V 3730 1550 50  0001 C CNN
 F 3 "~" H 3800 1550 50  0001 C CNN
@@
 P 3800 1950
 F 0 "R4" V 3593 1950 50  0000 C CNN
-F 1 "37" V 3684 1950 50  0000 C CNN
+F 1 "37 R" V 3684 1950 50  0000 C CNN
 F 2 "Resistor_SMD:R_0402_1005Metric" V 3730 1950 50  0001 C CNN
 F 3 "~" H 3800 1950 50  0001 C CNN
@@
 P 3800 2350
 F 0 "R5" V 3593 2350 50  0000 C CNN
-F 1 "37" V 3684 2350 50  0000 C CNN
+F 1 "37 R" V 3684 2350 50  0000 C CNN
 F 2 "Resistor_SMD:R_0402_1005Metric" V 3730 2350 50  0001 C CNN
 F 3 "~" H 3800 2350 50  0001 C CNN
@@
 P 6050 3850
 F 0 "C60" V 5798 3850 50  0000 C CNN
-F 1 "22µF 6,3V" V 5889 3850 50  0000 C CNN
+F 1 "22 µF 6,3V" V 5889 3850 50  0000 C CNN
 F 2 "Capacitor_SMD:C_1206_3216Metric" V 5900 3800 50  0001 C CNN
 F 3 "" H 6050 3850 50  0001 C CNN
@@
 Wire Wire Line
 	10300 4900 10400 4900
+Connection ~ 600  5150
+$Comp
+L power:GND #PWR?
+U 1 1 5BE33315
+P 800 4950
+F 0 "#PWR?" H 800 4700 50  0001 C CNN
+F 1 "GND" H 805 4777 50  0001 C CNN
+F 2 "" H 800 4950 50  0001 C CNN
+F 3 "" H 800 4950 50  0001 C CNN
+	1    800  4950
+	1    0    0    -1
+$EndComp
+Connection ~ 850  5900
+$Comp
+L power:GND #PWR?
+U 1 1 5BE9F8EF
+P 650 5700
+F 0 "#PWR?" H 650 5450 50  0001 C CNN
+F 1 "GND" H 655 5527 50  0001 C CNN
+F 2 "" H 650 5700 50  0001 C CNN
+F 3 "" H 650 5700 50  0001 C CNN
+	1    650  5700
+	0    -1   -1   0
+$EndComp
+Connection ~ 600  6600
+$Comp
+L power:GND #PWR?
+U 1 1 5BF0C4AF
+P 800 6400
+F 0 "#PWR?" H 800 6150 50  0001 C CNN
+F 1 "GND" H 805 6227 50  0001 C CNN
+F 2 "" H 800 6400 50  0001 C CNN
+F 3 "" H 800 6400 50  0001 C CNN
+	1    800  6400
+	1    0    0    -1
+$EndComp
+Connection ~ 850  7350
+$Comp
+L power:GND #PWR?
+U 1 1 5BF79106
+P 650 7150
+F 0 "#PWR?" H 650 6900 50  0001 C CNN
+F 1 "GND" H 655 6977 50  0001 C CNN
+F 2 "" H 650 7150 50  0001 C CNN
+F 3 "" H 650 7150 50  0001 C CNN
+	1    650  7150
+	0    -1   -1   0
+$EndComp
 $EndSCHEMATC

Commit message: a msg
Parts:
- Y6: footprint w_crystal:crystal_tc-38_horiz -> imm:Crystal_SMD_3215-2Pin_3.2x1.5mm
Connections:
- net UART2_RX: now also U1.202 (RX); no longer U1.111 (UART2_RX_/_PA01)
- net UART2_TX: now also U1.203 (TX); no longer U1.113 (UART2_TX_/_PA00)
- new net NIRQ: U1.113 (UART2_TX_/_PA00)
- new net NSEL: U1.111 (UART2_RX_/_PA01)
Changed lines of the file:
@@
 EESchema Schematic File Version 4
 LIBS:ass_shield-cache
-EELAYER 26 0
+EELAYER 29 0
 EELAYER END
 $Descr A4 11693 8268
 encoding utf-8
-Sheet 1 1
+Sheet 1 2
 Title ""
 Date ""
@@
 F 0 "Y6" V 5754 7481 50  0000 L CNN
 F 1 "16 MHz" V 5845 7481 50  0000 L CNN
-F 2 "w_crystal:crystal_tc-38_horiz" H 5800 7350 50  0001 C CNN
+F 2 "imm:Crystal_SMD_3215-2Pin_3.2x1.5mm" H 5800 7350 50  0001 C CNN
 F 3 "~" H 5800 7350 50  0001 C CNN
 	1    5800 7350
@@
 	0    -1   -1   0
 $EndComp
-Text GLabel 3100 1600 2    50   Input ~ 0
+Text GLabel 3100 800  2    50   Input ~ 0
 UART2_RX
-Text GLabel 3100 1700 2    50   Input ~ 0
+Text GLabel 3100 900  2    50   Input ~ 0
 UART2_TX
 Text GLabel 7250 3150 2    50   Input ~ 0
@@
 Connection ~ 600  5150
 $Comp
-L power:GND #PWR?
+L power:GND #PWR070
 U 1 1 5BE33315
 P 800 4950
-F 0 "#PWR?" H 800 4700 50  0001 C CNN
+F 0 "#PWR070" H 800 4700 50  0001 C CNN
 F 1 "GND" H 805 4777 50  0001 C CNN
 F 2 "" H 800 4950 50  0001 C CNN
@@
 Connection ~ 850  5900
 $Comp
-L power:GND #PWR?
+L power:GND #PWR063
 U 1 1 5BE9F8EF
 P 650 5700
-F 0 "#PWR?" H 650 5450 50  0001 C CNN
+F 0 "#PWR063" H 650 5450 50  0001 C CNN
 F 1 "GND" H 655 5527 50  0001 C CNN
 F 2 "" H 650 5700 50  0001 C CNN
@@
 Connection ~ 600  6600
 $Comp
-L power:GND #PWR?
+L power:GND #PWR071
 U 1 1 5BF0C4AF
 P 800 6400
-F 0 "#PWR?" H 800 6150 50  0001 C CNN
+F 0 "#PWR071" H 800 6150 50  0001 C CNN
 F 1 "GND" H 805 6227 50  0001 C CNN
 F 2 "" H 800 6400 50  0001 C CNN
@@
 Connection ~ 850  7350
 $Comp
-L power:GND #PWR?
+L power:GND #PWR069
 U 1 1 5BF79106
 P 650 7150
-F 0 "#PWR?" H 650 6900 50  0001 C CNN
+F 0 "#PWR069" H 650 6900 50  0001 C CNN
 F 1 "GND" H 655 6977 50  0001 C CNN
 F 2 "" H 650 7150 50  0001 C CNN
@@
 	0    -1   -1   0
 $EndComp
+$Sheet
+S 7350 6050 500  300
+U 5BE401CA
+F0 "list2" 50
+F1 "list2.sch" 50
+$EndSheet
+Text GLabel 3100 1600 2    50   Input ~ 0
+NSEL
+Text GLabel 3100 1700 2    50   Input ~ 0
+NIRQ
 $EndSCHEMATC

Commit message: a msg
Parts:
- C22, C32, C33, C34, C35, C40, C42, C44, C46, C49: value 0,1 µF -> 100 nF
- D24, D25, D26, D27: footprint imm:ADMP421 -> imm:ADMP421_2
Changed lines of the file:
@@
 P 10200 6250
 F 0 "C49" H 10085 6204 50  0000 R CNN
-F 1 "0,1 µF" H 10085 6295 50  0000 R CNN
+F 1 "100 nF" H 10085 6295 50  0000 R CNN
 F 2 "Capacitor_SMD:C_0402_1005Metric" V 10050 6200 50  0001 C CNN
 F 3 "" H 10200 6250 50  0001 C CNN
@@
 P 9800 6100
 F 0 "C46" H 9685 6054 50  0000 R CNN
-F 1 "0,1 µF" H 9685 6145 50  0000 R CNN
+F 1 "100 nF" H 9685 6145 50  0000 R CNN
 F 2 "Capacitor_SMD:C_0402_1005Metric" V 9650 6050 50  0001 C CNN
 F 3 "" H 9800 6100 50  0001 C CNN
@@
 P 9400 6250
 F 0 "C44" H 9285 6204 50  0000 R CNN
-F 1 "0,1 µF" H 9285 6295 50  0000 R CNN
+F 1 "100 nF" H 9285 6295 50  0000 R CNN
 F 2 "Capacitor_SMD:C_0402_1005Metric" V 9250 6200 50  0001 C CNN
 F 3 "" H 9400 6250 50  0001 C CNN
@@
 P 9000 6100
 F 0 "C42" H 8885 6054 50  0000 R CNN
-F 1 "0,1 µF" H 8885 6145 50  0000 R CNN
+F 1 "100 nF" H 8885 6145 50  0000 R CNN
 F 2 "Capacitor_SMD:C_0402_1005Metric" V 8850 6050 50  0001 C CNN
 F 3 "" H 9000 6100 50  0001 C CNN
@@
 P 8600 6250
 F 0 "C40" H 8485 6204 50  0000 R CNN
-F 1 "0,1 µF" H 8485 6295 50  0000 R CNN
+F 1 "100 nF" H 8485 6295 50  0000 R CNN
 F 2 "Capacitor_SMD:C_0402_1005Metric" V 8450 6200 50  0001 C CNN
 F 3 "" H 8600 6250 50  0001 C CNN
@@
 F 0 "D24" H 7550 4025 50  0000 C CNN
 F 1 "ADMP421" H 7550 3934 50  0000 C CNN
-F 2 "imm:ADMP421" H 7550 4050 50  0001 C CNN
+F 2 "imm:ADMP421_2" H 7550 4050 50  0001 C CNN
 F 3 "/home/user/kicad/libraries/imm_lib/ADMP421.pdf" H 7550 4050 50  0001 C CNN
 	1    7550 3800
@@
 F 0 "D25" H 7550 4575 50  0000 C CNN
 F 1 "ADMP421" H 7550 4484 50  0000 C CNN
-F 2 "imm:ADMP421" H 7550 4600 50  0001 C CNN
+F 2 "imm:ADMP421_2" H 7550 4600 50  0001 C CNN
 F 3 "/home/user/kicad/libraries/imm_lib/ADMP421.pdf" H 7550 4600 50  0001 C CNN
 	1    7550 4350
@@
 F 0 "D26" H 7550 5125 50  0000 C CNN
 F 1 "ADMP421" H 7550 5034 50  0000 C CNN
-F 2 "imm:ADMP421" H 7550 5150 50  0001 C CNN
+F 2 "imm:ADMP421_2" H 7550 5150 50  0001 C CNN
 F 3 "/home/user/kicad/libraries/imm_lib/ADMP421.pdf" H 7550 5150 50  0001 C CNN
 	1    7550 4900
@@
 F 0 "D27" H 7550 5675 50  0000 C CNN
 F 1 "ADMP421" H 7550 5584 50  0000 C CNN
-F 2 "imm:ADMP421" H 7550 5700 50  0001 C CNN
+F 2 "imm:ADMP421_2" H 7550 5700 50  0001 C CNN
 F 3 "/home/user/kicad/libraries/imm_lib/ADMP421.pdf" H 7550 5700 50  0001 C CNN
 	1    7550 5450
@@
 P 8050 4050
 F 0 "C32" H 8165 4096 50  0000 L CNN
-F 1 "0,1 µF" H 8165 4005 50  0000 L CNN
+F 1 "100 nF" H 8165 4005 50  0000 L CNN
 F 2 "Capacitor_SMD:C_0402_1005Metric" V 7900 4000 50  0001 C CNN
 F 3 "" H 8050 4050 50  0001 C CNN
@@
 P 8050 4600
 F 0 "C33" H 8165 4646 50  0000 L CNN
-F 1 "0,1 µF" H 8165 4555 50  0000 L CNN
+F 1 "100 nF" H 8165 4555 50  0000 L CNN
 F 2 "Capacitor_SMD:C_0402_1005Metric" V 7900 4550 50  0001 C CNN
 F 3 "" H 8050 4600 50  0001 C CNN
@@
 P 8050 5150
 F 0 "C34" H 8165 5196 50  0000 L CNN
-F 1 "0,1 µF" H 8165 5105 50  0000 L CNN
+F 1 "100 nF" H 8165 5105 50  0000 L CNN
 F 2 "Capacitor_SMD:C_0402_1005Metric" V 7900 5100 50  0001 C CNN
 F 3 "" H 8050 5150 50  0001 C CNN
@@
 P 8050 5700
 F 0 "C35" H 8165 5746 50  0000 L CNN
-F 1 "0,1 µF" H 8165 5655 50  0000 L CNN
+F 1 "100 nF" H 8165 5655 50  0000 L CNN
 F 2 "Capacitor_SMD:C_0402_1005Metric" V 7900 5650 50  0001 C CNN
 F 3 "" H 8050 5700 50  0001 C CNN
@@
 P 5300 3550
 F 0 "C22" V 5048 3550 50  0000 C CNN
-F 1 "0,1 µF" V 5139 3550 50  0000 C CNN
+F 1 "100 nF" V 5139 3550 50  0000 C CNN
 F 2 "Capacitor_SMD:C_0402_1005Metric" V 5150 3500 50  0001 C CNN
 F 3 "" H 5300 3550 50  0001 C CNN
