File: kicad/babana_pi_zero.kicad_pcb (KiCad board)
At the start: 2 copper layers, 73.3 x 73.3 mm, 6 parts, among them J1 RJ45, U1 OPiZero-imm_lib

Commit message: Add files via upload
Parts:
- added J2: i2s, Connector_PinHeader_2.54mm:PinHeader_1x03_P2.54mm_Vertical_SMD_Pin1Left, B.Cu at (159.7, 59.2)
- added J3: BananaPi/RaspberryPi, Button_Switch_SMD:SW_DIP_SPSTx04_Slide_KingTek_DSHP04TS_W7.62mm_P1.27mm, F.Cu at (167.5, 88.8)
- moved J1 49.1 mm to (140.7, 78.7)
Connections:
- D1 pad 12: (no net) -> Net-(D1-Pad12)
- D1 pad 18: (no net) -> IR
- D1 pad 26: (no net) -> PA10
- D1 pad 27: i2s_CLK -> Net-(D1-Pad27)
- D1 pad 28: i2s_WS -> Net-(D1-Pad28)
- D1 pad 35: PA10 -> Net-(D1-Pad35)
- D1 pad 38: (no net) -> i2s-DIN
- U1 pad 13: (no net) -> IR
Routing:
- net IR: track 0.00 -> 71.1 mm, vias 0 -> 1
- net Net-(D1-Pad44): track 17.6 -> 62.2 mm
- net Net-(D1-Pad35): track 0.00 -> 39.9 mm, vias 0 -> 2
- net Net-(D1-Pad45): track 23.0 -> 59.0 mm
- net i2s_CLK: track 8.57 -> 44.1 mm, vias 0 -> 3
- net i2s_WS: track 14.1 -> 44.0 mm, vias 0 -> 3
- net Net-(D1-Pad28): track 0.00 -> 27.1 mm, vias 0 -> 2
- net Net-(D1-Pad47): track 32.1 -> 57.7 mm
- net PA10: track 10.8 -> 33.3 mm
- net Net-(D1-Pad46): track 40.6 -> 62.4 mm
- net Net-(D1-Pad27): track 0.00 -> 21.8 mm, vias 0 -> 2
- net Net-(D1-Pad12): track 0.00 -> 13.0 mm
- net i2s-DIN: track 0.00 -> 7.84 mm, vias 0 -> 1
- net TX: track 50.6 -> 54.8 mm
- net RX: track 62.5 -> 63.3 mm
Other:
- board size 73.3 x 73.3 mm -> 60.4 x 71.5 mm
- board text added: "BananaPi Zero"
- board text added: "RaspberryPi Zero"
