File: kicad/nanopi_neo_core.kicad_pcb (KiCad board)
At the start: 2 copper layers, 49.8 x 62.6 mm, 8 parts, among them J1 HEADER-2x03, J2 RJ45, U1 OPiZero-imm_lib, X1 USB_F1

Commit message: Add files via upload
Parts:
- added J3: Conn_01x03_Male, Connector_PinHeader_2.54mm:PinHeader_1x03_P2.54mm_Vertical_SMD_Pin1Left, B.Cu at (157.1, 96.4)
Connections:
- D1 pad 111: (no net) -> Net-(D1-Pad111)
Routing:
- net Net-(D1-Pad111): track 0.00 -> 32.9 mm, vias 0 -> 1
- net Net-(D1-Pad109): track 21.2 -> 36.6 mm, vias 2 -> 4
- net Net-(D1-Pad108): track 24.9 -> 36.5 mm, vias 2 -> 5
- net Net-(D1-Pad110): track 26.7 -> 28.5 mm
