File: kicad/ass_shield (1-я копия).kicad_pcb (KiCad board)
At the start: 2 copper layers, 80 x 80 mm, 151 parts, among them J1 6-40V, J2 DEBUG, J3 5V, J4 UART2, J5 U.FL, J6 i2s, J7 SP, J8 U.FL, M1 CR1220SMD, Q1 BC817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

Commit message: a msg
Routing:
- net GND: track 177.8 -> 183.3 mm
- net Net-(D28-Pad7): track 12.0 -> 11.5 mm
