File: kicad/list2.sch (KiCad schematic (older format))
At the start: 27 parts, among them J9 Conn_Coaxial, U7 SI4432-B1-FMR, Y8 Crystal_GND24

Commit message: a msg
Parts:
- C61, C62: value 8.2pF -> 8,2 pF
- C63, C64: value 270pF -> 270 pF
- C65: value 10pF -> 10 pF
- C66, C73: value 0.1uF -> 100 nF
- C67: value 6.8pF -> 6,8 pF
- C68, C72: value 100pF -> 100 pF
- C69: value 12pF -> 12 pF
- C70: value 120pF -> 120 pF
- C71: value 33pF -> 33 pF
- C74: value 1uF -> 1 µF
- C75: value 4.7pF -> 4,7 pF
- L19: value 18nH -> 18 nH
- L20, L21: value 24nH -> 24 nH
- L22: value 11nH -> 11 nH
- L23: value 270nH -> 270 nH
- L24: value 33nH -> 33 nH
Changed lines of the file:
@@
 P 6350 2950
 F 0 "L23" H 6403 2988 39  0000 L CNN
-F 1 "270nH" H 6403 2913 39  0000 L CNN
+F 1 "270 nH" H 6403 2913 39  0000 L CNN
 F 2 "Inductor_SMD:L_0402_1005Metric" V 6200 2800 50  0001 C CNN
 F 3 "" H 6300 2950 50  0001 C CNN
@@
 P 5900 3150
 F 0 "C70" V 5648 3150 50  0000 C CNN
-F 1 "120pF" V 5739 3150 50  0000 C CNN
+F 1 "120 pF" V 5739 3150 50  0000 C CNN
 F 2 "Capacitor_SMD:C_0402_1005Metric" V 5750 3100 50  0001 C CNN
 F 3 "" H 5900 3150 50  0001 C CNN
@@
 P 5500 3150
 F 0 "L21" V 5666 3150 39  0000 C CNN
-F 1 "24nH" V 5591 3150 39  0000 C CNN
+F 1 "24 nH" V 5591 3150 39  0000 C CNN
 F 2 "Inductor_SMD:L_0402_1005Metric" V 5350 3000 50  0001 C CNN
 F 3 "" H 5450 3150 50  0001 C CNN
@@
 P 5100 3150
 F 0 "L20" V 5266 3150 39  0000 C CNN
-F 1 "24nH" V 5191 3150 39  0000 C CNN
+F 1 "24 nH" V 5191 3150 39  0000 C CNN
 F 2 "Inductor_SMD:L_0402_1005Metric" V 4950 3000 50  0001 C CNN
 F 3 "" H 5050 3150 50  0001 C CNN
@@
 P 5300 3450
 F 0 "C67" H 5185 3404 50  0000 R CNN
-F 1 "6.8pF" H 5185 3495 50  0000 R CNN
+F 1 "6,8 pF" H 5185 3495 50  0000 R CNN
 F 2 "Capacitor_SMD:C_0402_1005Metric" V 5150 3400 50  0001 C CNN
 F 3 "" H 5300 3450 50  0001 C CNN
@@
 P 4700 3150
 F 0 "C64" V 4448 3150 50  0000 C CNN
-F 1 "270pF" V 4539 3150 50  0000 C CNN
+F 1 "270 pF" V 4539 3150 50  0000 C CNN
 F 2 "Capacitor_SMD:C_0402_1005Metric" V 4550 3100 50  0001 C CNN
 F 3 "" H 4700 3150 50  0001 C CNN
@@
 P 5750 3550
 F 0 "C69" H 5635 3504 50  0000 R CNN
-F 1 "12pF" H 5635 3595 50  0000 R CNN
+F 1 "12 pF" H 5635 3595 50  0000 R CNN
 F 2 "Capacitor_SMD:C_0402_1005Metric" V 5600 3500 50  0001 C CNN
 F 3 "" H 5750 3550 50  0001 C CNN
@@
 P 6100 3550
 F 0 "L22" H 6153 3588 39  0000 L CNN
-F 1 "11nH" H 6153 3513 39  0000 L CNN
+F 1 "11 nH" H 6153 3513 39  0000 L CNN
 F 2 "Inductor_SMD:L_0402_1005Metric" V 5950 3400 50  0001 C CNN
 F 3 "" H 6050 3550 50  0001 C CNN
@@
 P 9600 3300
 F 0 "L24" H 9653 3338 39  0000 L CNN
-F 1 "33nH" H 9653 3263 39  0000 L CNN
+F 1 "33 nH" H 9653 3263 39  0000 L CNN
 F 2 "Inductor_SMD:L_0402_1005Metric" V 9450 3150 50  0001 C CNN
 F 3 "" H 9550 3300 50  0001 C CNN
@@
 P 9600 3600
 F 0 "C75" H 9485 3554 50  0000 R CNN
-F 1 "4.7pF" H 9485 3645 50  0000 R CNN
+F 1 "4,7 pF" H 9485 3645 50  0000 R CNN
 F 2 "Capacitor_SMD:C_0402_1005Metric" V 9450 3550 50  0001 C CNN
 F 3 "" H 9600 3600 50  0001 C CNN
@@
 P 2650 3550
 F 0 "L19" V 2816 3550 39  0000 C CNN
-F 1 "18nH" V 2741 3550 39  0000 C CNN
+F 1 "18 nH" V 2741 3550 39  0000 C CNN
 F 2 "Inductor_SMD:L_0402_1005Metric" V 2500 3400 50  0001 C CNN
 F 3 "" H 2600 3550 50  0001 C CNN
@@
 P 3100 3550
 F 0 "C63" V 2848 3550 50  0000 C CNN
-F 1 "270pF" V 2939 3550 50  0000 C CNN
+F 1 "270 pF" V 2939 3550 50  0000 C CNN
 F 2 "Capacitor_SMD:C_0402_1005Metric" V 2950 3500 50  0001 C CNN
 F 3 "" H 3100 3550 50  0001 C CNN
@@
 P 2900 3950
 F 0 "C62" H 2785 3904 50  0000 R CNN
-F 1 "8.2pF" H 2785 3995 50  0000 R CNN
+F 1 "8,2 pF" H 2785 3995 50  0000 R CNN
 F 2 "Capacitor_SMD:C_0402_1005Metric" V 2750 3900 50  0001 C CNN
 F 3 "" H 2900 3950 50  0001 C CNN
@@
 P 2450 3950
 F 0 "C61" H 2335 3904 50  0000 R CNN
-F 1 "8.2pF" H 2335 3995 50  0000 R CNN
+F 1 "8,2 pF" H 2335 3995 50  0000 R CNN
 F 2 "Capacitor_SMD:C_0402_1005Metric" V 2300 3900 50  0001 C CNN
 F 3 "" H 2450 3950 50  0001 C CNN
@@
 P 6000 2400
 F 0 "C71" H 5885 2354 50  0000 R CNN
-F 1 "33pF" H 5885 2445 50  0000 R CNN
+F 1 "33 pF" H 5885 2445 50  0000 R CNN
 F 2 "Capacitor_SMD:C_0402_1005Metric" V 5850 2350 50  0001 C CNN
 F 3 "" H 6000 2400 50  0001 C CNN
@@
 P 5550 2400
 F 0 "C68" H 5435 2354 50  0000 R CNN
-F 1 "100pF" H 5435 2445 50  0000 R CNN
+F 1 "100 pF" H 5435 2445 50  0000 R CNN
 F 2 "Capacitor_SMD:C_0402_1005Metric" V 5400 2350 50  0001 C CNN
 F 3 "" H 5550 2400 50  0001 C CNN
@@
 P 5100 2400
 F 0 "C66" H 4985 2354 50  0000 R CNN
-F 1 "0.1uF" H 4985 2445 50  0000 R CNN
+F 1 "100 nF" H 4985 2445 50  0000 R CNN
 F 2 "Capacitor_SMD:C_0402_1005Metric" V 4950 2350 50  0001 C CNN
 F 3 "" H 5100 2400 50  0001 C CNN
@@
 P 6950 3600
 F 0 "C74" H 6835 3554 50  0000 R CNN
-F 1 "1uF" H 6835 3645 50  0000 R CNN
+F 1 "1 µF" H 6835 3645 50  0000 R CNN
 F 2 "Capacitor_SMD:C_0402_1005Metric" V 6800 3550 50  0001 C CNN
 F 3 "" H 6950 3600 50  0001 C CNN
@@
 P 6450 3600
 F 0 "C72" H 6335 3554 50  0000 R CNN
-F 1 "100pF" H 6335 3645 50  0000 R CNN
+F 1 "100 pF" H 6335 3645 50  0000 R CNN
 F 2 "Capacitor_SMD:C_0402_1005Metric" V 6300 3550 50  0001 C CNN
 F 3 "" H 6450 3600 50  0001 C CNN
@@
 P 4700 4000
 F 0 "C65" V 4448 4000 50  0000 C CNN
-F 1 "10pF" V 4539 4000 50  0000 C CNN
+F 1 "10 pF" V 4539 4000 50  0000 C CNN
 F 2 "Capacitor_SMD:C_0402_1005Metric" V 4550 3950 50  0001 C CNN
 F 3 "" H 4700 4000 50  0001 C CNN
@@
 P 6750 2500
 F 0 "C73" H 6635 2454 50  0000 R CNN
-F 1 "0.1uF" H 6635 2545 50  0000 R CNN
+F 1 "100 nF" H 6635 2545 50  0000 R CNN
 F 2 "Capacitor_SMD:C_0402_1005Metric" V 6600 2450 50  0001 C CNN
 F 3 "" H 6750 2500 50  0001 C CNN
